File: Termostato/schema.sch (EAGLE design)
At the start: 5 parts, among them K1 RELAY-SPDT-JZC-11F

Commit message: Updated schematics V1.1
Connections:
- new net 3.3V: B1.3.3V, U$1.CH_PD, U$1.VCC
- net RX: now also B1.D2; no longer B1.*D3
- net TX: now also B1.*D3; no longer B1.D2
- net VCC: no longer U$1.VCC
Changed lines of the file:
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@@
 <part name="GND3" library="SparkFun-PowerSymbols" deviceset="GND" device=""/>
 <part name="GND4" library="SparkFun-PowerSymbols" deviceset="GND" device=""/>
-<part name="P+1" library="supply1" library_urn="urn:adsk.eagle:library:371" deviceset="VCC" device=""/>
 <part name="P+2" library="supply1" library_urn="urn:adsk.eagle:library:371" deviceset="VCC" device=""/>
 <part name="P+3" library="supply1" library_urn="urn:adsk.eagle:library:371" deviceset="VCC" device=""/>
@@
 <instance part="GND3" gate="1" x="106.68" y="104.14" rot="R270"/>
 <instance part="GND4" gate="1" x="48.26" y="106.68" rot="R270"/>
-<instance part="P+1" gate="VCC" x="106.68" y="86.36" rot="R90"/>
 <instance part="P+2" gate="VCC" x="104.14" y="134.62" rot="R90"/>
 <instance part="P+3" gate="VCC" x="48.26" y="121.92" rot="R90"/>
@@
 <wire x1="106.68" y1="134.62" x2="121.92" y2="134.62" width="0.1524" layer="91"/>
 </segment>
-<segment>
-<pinref part="P+1" gate="VCC" pin="VCC"/>
-<pinref part="U$1" gate="G$1" pin="VCC"/>
-<wire x1="109.22" y1="86.36" x2="116.84" y2="86.36" width="0.1524" layer="91"/>
-</segment>
 </net>
 <net name="N$3" class="0">
@@
 </segment>
 <segment>
-<pinref part="B1" gate="G$1" pin="D2"/>
-<wire x1="83.82" y1="139.7" x2="86.36" y2="139.7" width="0.1524" layer="91"/>
-<label x="86.36" y="139.7" size="1.778" layer="95"/>
+<pinref part="B1" gate="G$1" pin="*D3"/>
+<wire x1="83.82" y1="137.16" x2="86.36" y2="137.16" width="0.1524" layer="91"/>
+<label x="86.36" y="137.16" size="1.778" layer="95"/>
 </segment>
 </net>
@@
 </segment>
 <segment>
-<pinref part="B1" gate="G$1" pin="*D3"/>
-<wire x1="83.82" y1="137.16" x2="86.36" y2="137.16" width="0.1524" layer="91"/>
-<label x="86.36" y="137.16" size="1.778" layer="95"/>
+<pinref part="B1" gate="G$1" pin="D2"/>
+<wire x1="83.82" y1="139.7" x2="86.36" y2="139.7" width="0.1524" layer="91"/>
+<label x="86.36" y="139.7" size="1.778" layer="95"/>
 </segment>
 </net>
+<net name="3.3V" class="0">
+<segment>
+<pinref part="U$1" gate="G$1" pin="VCC"/>
+<wire x1="114.3" y1="86.36" x2="116.84" y2="86.36" width="0.1524" layer="91"/>
+<label x="111.76" y="86.36" size="1.778" layer="95"/>
+</segment>
+<segment>
+<pinref part="B1" gate="G$1" pin="3.3V"/>
+<wire x1="58.42" y1="116.84" x2="55.88" y2="116.84" width="0.1524" layer="91"/>
+<label x="53.34" y="116.84" size="1.778" layer="95"/>
+</segment>
+<segment>
+<pinref part="U$1" gate="G$1" pin="CH_PD"/>
+<wire x1="116.84" y1="96.52" x2="114.3" y2="96.52" width="0.1524" layer="91"/>
+<label x="111.76" y="96.52" size="1.778" layer="95"/>
+</segment>
+</net>

Commit message: Updated schematic
Parts:
- added LCD1: LCD-16X2SILK, SparkFun-Displays:LCD-16X2SILK
- added R1, R2: 220, SparkFun-Resistors:220OHM-0603-1/10W-1%
- added S2, S3: (no value), SparkFun-Retired:TAC_SWITCHPTH
- added VR1: 10k, SparkFun-Resistors:TRIMPOT-SMD-3MM-OPEN-1/10W-25%
Connections:
- new net D10: B1.*D10, LCD1.DB5
- new net D11: B1.*D11, LCD1.DB6
- new net D12: B1.D12, LCD1.DB7
- new net D13: B1.D13, K1.COIL2
- new net D4: B1.D4, S2.4
- new net D5: B1.*D5, S3.4
- new net D8: B1.D8, LCD1.E
- new net D9: B1.*D9, LCD1.DB4
- new net N$1: LCD1.VO, VR1.WIPER
- new net N$2: R2.1, S2.3
- new net N$4: R1.1, S3.3
- new net N$5: S3.1
- net D7: now also LCD1.RS; no longer K1.COIL2
- net GND: now also LCD1.K, LCD1.R/W, LCD1.VDD, R1.2, R2.2, VR1.CCW
- net VCC: now also LCD1.A, LCD1.VSS, S2.1, VR1.CW
Other:
- moved on the sheet: K1

Commit message: Arduino shield
Parts:
- B1: value ARDUINO_UNO_R3NO_HOLES -> ARDUINO_UNO_R3_SHIELDBASIC; device SparkFun-Boards:ARDUINO_UNO_R3NO_HOLES -> SparkFun-Boards:ARDUINO_UNO_R3_SHIELDBASIC
Connections:
- net 3.3V: no longer B1.3.3V
Changed lines of the file:
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@@
 <layers>
 <layer number="1" name="Top" color="4" fill="1" visible="no" active="no"/>
+<layer number="2" name="Route2" color="1" fill="3" visible="no" active="no"/>
+<layer number="3" name="Route3" color="4" fill="3" visible="no" active="no"/>
+<layer number="4" name="Route4" color="1" fill="4" visible="no" active="no"/>
+<layer number="5" name="Route5" color="4" fill="4" visible="no" active="no"/>
+<layer number="6" name="Route6" color="1" fill="8" visible="no" active="no"/>
+<layer number="7" name="Route7" color="4" fill="8" visible="no" active="no"/>
+<layer number="8" name="Route8" color="1" fill="2" visible="no" active="no"/>
+<layer number="9" name="Route9" color="4" fill="2" visible="no" active="no"/>
+<layer number="10" name="Route10" color="1" fill="7" visible="no" active="no"/>
+<layer number="11" name="Route11" color="4" fill="7" visible="no" active="no"/>
+<layer number="12" name="Route12" color="1" fill="5" visible="no" active="no"/>
+<layer number="13" name="Route13" color="4" fill="5" visible="no" active="no"/>
+<layer number="14" name="Route14" color="1" fill="6" visible="no" active="no"/>
+<layer number="15" name="Route15" color="4" fill="6" visible="no" active="no"/>
 <layer number="16" name="Bottom" color="1" fill="1" visible="no" active="no"/>
 <layer number="17" name="Pads" color="2" fill="1" visible="no" active="no"/>
@@
 </classes>
 <parts>
-<part name="B1" library="SparkFun-Boards" deviceset="ARDUINO_UNO_R3" device="NO_HOLES"/>
 <part name="K1" library="SparkFun-Electromechanical" deviceset="RELAY-SPDT" device="-JZC-11F"/>
 <part name="U1" library="RHT03_DHT-22_AM2302" deviceset="RHT03_DHT-22_AM2302" device="RA"/>
@@
 <part name="P+6" library="supply1" library_urn="urn:adsk.eagle:library:371" deviceset="VCC" device=""/>
 <part name="P+7" library="supply1" library_urn="urn:adsk.eagle:library:371" deviceset="VCC" device=""/>
+<part name="B1" library="SparkFun-Boards" deviceset="ARDUINO_UNO_R3_SHIELD" device="BASIC"/>
 </parts>
 <sheets>
@@
 </plain>
 <instances>
-<instance part="B1" gate="G$1" x="71.12" y="116.84"/>
 <instance part="K1" gate="K$1" x="2.54" y="142.24" rot="R180"/>
 <instance part="U1" gate="G$1" x="132.08" y="127"/>
@@
 <instance part="P+6" gate="VCC" x="96.52" y="152.4" rot="R90"/>
 <instance part="P+7" gate="VCC" x="96.52" y="165.1" rot="R90"/>
+<instance part="B1" gate="G$1" x="71.12" y="129.54"/>
 </instances>
 <busses>
@@
 <segment>
 <pinref part="GND4" gate="1" pin="GND"/>
+<wire x1="50.8" y1="106.68" x2="58.42" y2="106.68" width="0.1524" layer="91"/>
 <pinref part="B1" gate="G$1" pin="GND@0"/>
-<wire x1="50.8" y1="106.68" x2="58.42" y2="106.68" width="0.1524" layer="91"/>
 </segment>
 <segment>
@@
 <segment>
 <pinref part="P+3" gate="VCC" pin="VCC"/>
+<wire x1="50.8" y1="121.92" x2="58.42" y2="121.92" width="0.1524" layer="91"/>
 <pinref part="B1" gate="G$1" pin="VIN"/>
-<wire x1="50.8" y1="121.92" x2="58.42" y2="121.92" width="0.1524" layer="91"/>
 </segment>
 <segment>
@@
 <net name="N$3" class="0">
 <segment>
-<pinref part="B1" gate="G$1" pin="*D6"/>
 <pinref part="U1" gate="G$1" pin="DATA"/>
 <wire x1="83.82" y1="129.54" x2="121.92" y2="129.54" width="0.1524" layer="91"/>
+<pinref part="B1" gate="G$1" pin="*D6"/>
 </segment>
 </net>
 <net name="D7" class="0">
 <segment>
-<pinref part="B1" gate="G$1" pin="D7"/>
 <wire x1="83.82" y1="127" x2="86.36" y2="127" width="0.1524" layer="91"/>
 <label x="83.82" y="127" size="1.778" layer="95"/>
+<pinref part="B1" gate="G$1" pin="D7"/>
 </segment>
 <segment>
@@
 </segment>
 <segment>
-<pinref part="B1" gate="G$1" pin="*D3"/>
 <wire x1="83.82" y1="137.16" x2="86.36" y2="137.16" width="0.1524" layer="91"/>
 <label x="83.82" y="137.16" size="1.778" layer="95"/>
+<pinref part="B1" gate="G$1" pin="*D3"/>
 </segment>
 </net>
@@
 </segment>
 <segment>
-<pinref part="B1" gate="G$1" pin="D2"/>
 <wire x1="83.82" y1="139.7" x2="86.36" y2="139.7" width="0.1524" layer="91"/>
 <label x="83.82" y="139.7" size="1.778" layer="95"/>
+<pinref part="B1" gate="G$1" pin="D2"/>
 </segment>
 </net>
@@
 </segment>
 <segment>
-<pinref part="B1" gate="G$1" pin="3.3V"/>
-<wire x1="58.42" y1="116.84" x2="55.88" y2="116.84" width="0.1524" layer="91"/>
-<label x="53.34" y="116.84" size="1.778" layer="95"/>
-</segment>
-<segment>
 <pinref part="U$1" gate="G$1" pin="CH_PD"/>
 <wire x1="116.84" y1="96.52" x2="114.3" y2="96.52" width="0.1524" layer="91"/>
@@
 <segment>
 <pinref part="B1" gate="G$1" pin="D13"/>
-<wire x1="83.82" y1="109.22" x2="86.36" y2="109.22" width="0.1524" layer="91"/>
-<label x="83.82" y="109.22" size="1.778" layer="95"/>
+<wire x1="83.82" y1="111.76" x2="86.36" y2="111.76" width="0.1524" layer="91"/>
+<label x="83.82" y="111.76" size="1.778" layer="95"/>
 </segment>
 </net>
@@
 <segment>
 <pinref part="B1" gate="G$1" pin="D8"/>
-<wire x1="83.82" y1="121.92" x2="86.36" y2="121.92" width="0.1524" layer="91"/>
-<label x="83.82" y="121.92" size="1.778" layer="95"/>
+<wire x1="83.82" y1="124.46" x2="86.36" y2="124.46" width="0.1524" layer="91"/>
+<label x="83.82" y="124.46" size="1.778" layer="95"/>
 </segment>
 </net>
@@
 <segment>
 <pinref part="B1" gate="G$1" pin="*D9"/>
-<wire x1="83.82" y1="119.38" x2="86.36" y2="119.38" width="0.1524" layer="91"/>
-<label x="83.82" y="119.38" size="1.778" layer="95"/>
+<wire x1="83.82" y1="121.92" x2="86.36" y2="121.92" width="0.1524" layer="91"/>
+<label x="83.82" y="121.92" size="1.778" layer="95"/>
 </segment>
 </net>
@@
 <segment>
 <pinref part="B1" gate="G$1" pin="*D10"/>
-<wire x1="83.82" y1="116.84" x2="86.36" y2="116.84" width="0.1524" layer="91"/>
-<label x="83.82" y="116.84" size="1.778" layer="95"/>
+<wire x1="83.82" y1="119.38" x2="86.36" y2="119.38" width="0.1524" layer="91"/>
+<label x="83.82" y="119.38" size="1.778" layer="95"/>
 </segment>
 </net>
@@
 <segment>
 <pinref part="B1" gate="G$1" pin="*D11"/>
-<wire x1="83.82" y1="114.3" x2="86.36" y2="114.3" width="0.1524" layer="91"/>
-<label x="83.82" y="114.3" size="1.778" layer="95"/>
+<wire x1="83.82" y1="116.84" x2="86.36" y2="116.84" width="0.1524" layer="91"/>
+<label x="83.82" y="116.84" size="1.778" layer="95"/>
 </segment>
 </net>
@@
 <segment>
 <pinref part="B1" gate="G$1" pin="D12"/>
-<wire x1="83.82" y1="111.76" x2="86.36" y2="111.76" width="0.1524" layer="91"/>
-<label x="83.82" y="111.76" size="1.778" layer="95"/>
+<wire x1="83.82" y1="114.3" x2="86.36" y2="114.3" width="0.1524" layer="91"/>
+<label x="83.82" y="114.3" size="1.778" layer="95"/>
 </segment>
 </net>
@@
 </segment>
 <segment>
-<pinref part="B1" gate="G$1" pin="D4"/>
 <wire x1="83.82" y1="134.62" x2="86.36" y2="134.62" width="0.1524" layer="91"/>
 <label x="83.82" y="134.62" size="1.778" layer="95"/>
+<pinref part="B1" gate="G$1" pin="D4"/>
 </segment>
 </net>
@@
 </segment>
 <segment>
-<pinref part="B1" gate="G$1" pin="*D5"/>
 <wire x1="83.82" y1="132.08" x2="86.36" y2="132.08" width="0.1524" layer="91"/>
 <label x="83.82" y="132.08" size="1.778" layer="95"/>
-</segment>
-</net>
+<pinref part="B1" gate="G$1" pin="*D5"/>
+</segment>
+</net>

Commit message: Update schematics: add 3.3V connection and switch from VIN to 5V
Connections:
- net 3.3V: now also B1.3.3V
- net VCC: now also B1.5V; no longer B1.VIN
Changed lines of the file:
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@@
 <instance part="GND4" gate="1" x="48.26" y="106.68" rot="R270"/>
 <instance part="P+2" gate="VCC" x="104.14" y="134.62" rot="R90"/>
-<instance part="P+3" gate="VCC" x="48.26" y="121.92" rot="R90"/>
+<instance part="P+3" gate="VCC" x="35.56" y="119.38" rot="R90"/>
 <instance part="LCD1" gate="G$1" x="2.54" y="101.6" rot="R180"/>
 <instance part="GND5" gate="1" x="25.4" y="119.38" rot="R90"/>
@@
 <net name="VCC" class="0">
 <segment>
-<pinref part="P+3" gate="VCC" pin="VCC"/>
-<wire x1="50.8" y1="121.92" x2="58.42" y2="121.92" width="0.1524" layer="91"/>
-<pinref part="B1" gate="G$1" pin="VIN"/>
-</segment>
-<segment>
 <pinref part="P+2" gate="VCC" pin="VCC"/>
 <pinref part="U1" gate="G$1" pin="VDD"/>
@@
 <wire x1="104.14" y1="165.1" x2="99.06" y2="165.1" width="0.1524" layer="91"/>
 <pinref part="P+7" gate="VCC" pin="VCC"/>
+</segment>
+<segment>
+<pinref part="P+3" gate="VCC" pin="VCC"/>
+<pinref part="B1" gate="G$1" pin="5V"/>
+<wire x1="38.1" y1="119.38" x2="58.42" y2="119.38" width="0.1524" layer="91"/>
 </segment>
 </net>
@@
 <label x="111.76" y="96.52" size="1.778" layer="95"/>
 </segment>
+<segment>
+<label x="50.8" y="83.82" size="1.778" layer="95"/>
+</segment>
+<segment>
+<pinref part="B1" gate="G$1" pin="3.3V"/>
+<wire x1="58.42" y1="116.84" x2="48.26" y2="116.84" width="0.1524" layer="91"/>
+<label x="48.26" y="116.84" size="1.778" layer="95"/>
+</segment>
 </net>

Commit message: Updated board design
Parts:
- removed R1, R2: 220, SparkFun-Resistors:220OHM-0603-1/10W-1%
- removed VR1: 10k, SparkFun-Resistors:TRIMPOT-SMD-3MM-OPEN-1/10W-25%
- added R3, R4: 220, resistor:R-EU_0204/7
Connections:
- removed net N$1: LCD1.VO, VR1.WIPER
- net GND: now also R3.2, R4.2; no longer R1.2, R2.2, VR1.CCW
- net N$2: now also R3.1; no longer R2.1
- net N$4: now also R4.1; no longer R1.1
- net VCC: no longer VR1.CW
Changed lines of the file:
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@@
 <?xml version="1.0" encoding="utf-8"?>
 <!DOCTYPE eagle SYSTEM "eagle.dtd">
-<eagle version="8.4.0">
+<eagle version="7.7.0">
 <drawing>
 <settings>
@@
 <part name="GND3" library="SparkFun-PowerSymbols" deviceset="GND" device=""/>
 <part name="GND4" library="SparkFun-PowerSymbols" deviceset="GND" device=""/>
-<part name="P+2" library="supply1" library_urn="urn:adsk.eagle:library:371" deviceset="VCC" device=""/>
-<part name="P+3" library="supply1" library_urn="urn:adsk.eagle:library:371" deviceset="VCC" device=""/>
+<part name="P+2" library="supply1" deviceset="VCC" device=""/>
+<part name="P+3" library="supply1" deviceset="VCC" device=""/>
 <part name="LCD1" library="SparkFun-Displays" deviceset="LCD-16X2" device="SILK"/>
 <part name="GND5" library="SparkFun-PowerSymbols" deviceset="GND" device=""/>
 <part name="GND6" library="SparkFun-PowerSymbols" deviceset="GND" device=""/>
-<part name="P+1" library="supply1" library_urn="urn:adsk.eagle:library:371" deviceset="VCC" device=""/>
+<part name="P+1" library="supply1" deviceset="VCC" device=""/>
 <part name="GND7" library="SparkFun-PowerSymbols" deviceset="GND" device=""/>
-<part name="VR1" library="SparkFun-Resistors" deviceset="TRIMPOT" device="-SMD-3MM-OPEN-1/10W-25%" value="10k"/>
-<part name="P+4" library="supply1" library_urn="urn:adsk.eagle:library:371" deviceset="VCC" device=""/>
-<part name="GND8" library="SparkFun-PowerSymbols" deviceset="GND" device=""/>
-<part name="P+5" library="supply1" library_urn="urn:adsk.eagle:library:371" deviceset="VCC" device=""/>
+<part name="P+5" library="supply1" deviceset="VCC" device=""/>
 <part name="S2" library="SparkFun-Retired" deviceset="TAC_SWITCH" device="PTH"/>
 <part name="S3" library="SparkFun-Retired" deviceset="TAC_SWITCH" device="PTH"/>
-<part name="R1" library="SparkFun-Resistors" deviceset="220OHM" device="-0603-1/10W-1%" value="220"/>
-<part name="R2" library="SparkFun-Resistors" deviceset="220OHM" device="-0603-1/10W-1%" value="220"/>
 <part name="GND9" library="SparkFun-PowerSymbols" deviceset="GND" device=""/>
 <part name="GND10" library="SparkFun-PowerSymbols" deviceset="GND" device=""/>
-<part name="P+6" library="supply1" library_urn="urn:adsk.eagle:library:371" deviceset="VCC" device=""/>
-<part name="P+7" library="supply1" library_urn="urn:adsk.eagle:library:371" deviceset="VCC" device=""/>
+<part name="P+6" library="supply1" deviceset="VCC" device=""/>
+<part name="P+7" library="supply1" deviceset="VCC" device=""/>
 <part name="B1" library="SparkFun-Boards" deviceset="ARDUINO_UNO_R3_SHIELD" device="BASIC"/>
+<part name="R3" library="resistor" deviceset="R-EU_" device="0204/7" value="220"/>
+<part name="R4" library="resistor" deviceset="R-EU_" device="0204/7" value="220"/>
 </parts>
 <sheets>
@@
 <instance part="P+1" gate="VCC" x="25.4" y="76.2" rot="R180"/>
 <instance part="GND7" gate="1" x="25.4" y="91.44" rot="R90"/>
-<instance part="VR1" gate="R?" x="35.56" y="86.36" rot="R180"/>
-<instance part="P+4" gate="VCC" x="35.56" y="96.52"/>
-<instance part="GND8" gate="1" x="35.56" y="76.2"/>
 <instance part="P+5" gate="VCC" x="20.32" y="114.3" rot="R180"/>
 <instance part="S2" gate="S" x="109.22" y="165.1"/>
 <instance part="S3" gate="S" x="109.22" y="152.4"/>
-<instance part="R1" gate="G$1" x="124.46" y="152.4"/>
-<instance part="R2" gate="G$1" x="124.46" y="165.1"/>
 <instance part="GND9" gate="1" x="137.16" y="165.1" rot="R90"/>
 <instance part="GND10" gate="1" x="137.16" y="152.4" rot="R90"/>
@@
 <instance part="P+7" gate="VCC" x="96.52" y="165.1" rot="R90"/>
 <instance part="B1" gate="G$1" x="71.12" y="129.54"/>
+<instance part="R3" gate="G$1" x="124.46" y="165.1"/>
+<instance part="R4" gate="G$1" x="124.46" y="152.4"/>
 </instances>
 <busses>
@@
 </segment>
 <segment>
-<pinref part="VR1" gate="R?" pin="CCW"/>
-<pinref part="GND8" gate="1" pin="GND"/>
-<wire x1="35.56" y1="81.28" x2="35.56" y2="78.74" width="0.1524" layer="91"/>
-</segment>
-<segment>
 <pinref part="GND10" gate="1" pin="GND"/>
-<pinref part="R1" gate="G$1" pin="2"/>
 <wire x1="134.62" y1="152.4" x2="129.54" y2="152.4" width="0.1524" layer="91"/>
+<pinref part="R4" gate="G$1" pin="2"/>
 </segment>
 <segment>
 <pinref part="GND9" gate="1" pin="GND"/>
-<pinref part="R2" gate="G$1" pin="2"/>
 <wire x1="134.62" y1="165.1" x2="129.54" y2="165.1" width="0.1524" layer="91"/>
+<pinref part="R3" gate="G$1" pin="2"/>
 </segment>
 </net>
@@
 </segment>
 <segment>
-<pinref part="P+4" gate="VCC" pin="VCC"/>
-<pinref part="VR1" gate="R?" pin="CW"/>
-<wire x1="35.56" y1="93.98" x2="35.56" y2="91.44" width="0.1524" layer="91"/>
-</segment>
-<segment>
 <pinref part="LCD1" gate="G$1" pin="A"/>
 <pinref part="P+5" gate="VCC" pin="VCC"/>
@@
 </segment>
 <segment>
-<label x="50.8" y="83.82" size="1.778" layer="95"/>
-</segment>
-<segment>
 <pinref part="B1" gate="G$1" pin="3.3V"/>
 <wire x1="58.42" y1="116.84" x2="48.26" y2="116.84" width="0.1524" layer="91"/>
@@
 </segment>
 </net>
-<net name="N$1" class="0">
-<segment>
-<pinref part="LCD1" gate="G$1" pin="VO"/>
-<pinref part="VR1" gate="R?" pin="WIPER"/>
-<wire x1="12.7" y1="86.36" x2="30.48" y2="86.36" width="0.1524" layer="91"/>
-</segment>
-</net>
 <net name="D13" class="0">
 <segment>
@@
 <net name="N$2" class="0">
 <segment>
-<pinref part="R2" gate="G$1" pin="1"/>
 <pinref part="S2" gate="S" pin="3"/>
 <wire x1="119.38" y1="165.1" x2="114.3" y2="165.1" width="0.1524" layer="91"/>
+<pinref part="R3" gate="G$1" pin="1"/>
 </segment>
 </net>
 <net name="N$4" class="0">
 <segment>
-<pinref part="R1" gate="G$1" pin="1"/>
 <pinref part="S3" gate="S" pin="3"/>
 <wire x1="119.38" y1="152.4" x2="114.3" y2="152.4" width="0.1524" layer="91"/>
+<pinref part="R4" gate="G$1" pin="1"/>
 </segment>
 </net>
@@
 </schematic>
 </drawing>
-<compatibility>
-<note version="8.2" severity="warning">
-Since Version 8.2, EAGLE supports online libraries. The ids
-of those online libraries will not be understood (or retained)
-with this version.
-</note>
-<note version="8.3" severity="warning">
-Since Version 8.3, EAGLE supports URNs for individual library
-assets (packages, symbols, and devices). The URNs of those assets
-will not be understood (or retained) with this version.
-</note>
-</compatibility>
 </eagle>
